Commit message: mjcf와 방향 통일

File: Industrial_Safety_Patrol/urdf/turtlebot_patrol.urdf (robot description, URDF)
Before this commit: robot turtlebot_patrol, 9 links, 8 joints
Joints:
- joint lidar_joint: origin xyz=0 0 0.107 rpy=0 0 0 -> xyz=0.07 0 0.107 rpy=0 0 0

Commit message: align with mjcf

File: Industrial_Safety_Patrol/urdf/turtlebot_patrol.urdf (robot description, URDF)
Before this commit: robot turtlebot_patrol, 9 links, 8 joints
Links:
- link base_link: mass 0.7 -> 0.85; geometry collision box size=0.138 0.150 0.005; collision box size=0.138 0.150 0.005
- link camera_link: mass 0.03 -> 0.02; geometry visual box size=0.024 0.070 0.020
- link caster_ball_link: mass 0.02 -> 0.01; geometry collision sphere radius=0.010; visual sphere radius=0.010
- link imu_link: mass None -> 0.001
- link lidar_link: mass 0.1 -> 0.08; geometry visual cylinder length=0.024 radius=0.035
- link sensor_tower_link: geometry visual cylinder length=0.03 radius=0.008
- link wheel_left_link: mass 0.05 -> 0.04; geometry collision cylinder length=0.018 radius=0.033; visual cylinder length=0.018 radius=0.033
- link wheel_right_link: mass 0.05 -> 0.04; geometry collision cylinder length=0.018 radius=0.033; visual cylinder length=0.018 radius=0.033
Joints:
- joint base_joint: origin xyz=0 0 0.043 rpy=0 0 0 -> xyz=0 0 0.033 rpy=0 0 0
- joint camera_joint: origin xyz=0.069 0 0.06 rpy=0 0 0 -> xyz=-0.05 0 0.2125 rpy=0 0 0
- joint caster_joint: origin xyz=-0.06 0 -0.023 rpy=0 0 0 -> xyz=-0.055 0 -0.023 rpy=0 0 0
- joint imu_joint: origin xyz=0 0 0.01 rpy=0 0 0 -> xyz=0 0 0.005 rpy=0 0 0
- joint lidar_joint: origin xyz=0.07 0 0.107 rpy=0 0 0 -> xyz=0 0 0.030 rpy=0 0 0
- joint sensor_tower_joint: origin xyz=0 0 0.055 rpy=0 0 0 -> xyz=0 0 0.1375 rpy=0 0 0
