Commit message: add mimic for tf

File: cobot_pnp_safety/urdf/ur5e_2f85.urdf (robot description, URDF)
Before this commit: robot ur5e_2f85, 24 links, 23 joints
Links:
- removed link 2f85_base
- removed link base_mount
- removed link left_coupler
- removed link left_driver
- removed link left_follower
- removed link left_pad
- removed link left_silicone_pad
- removed link left_spring_link
- removed link pinch_site
- removed link right_coupler
- removed link right_driver
- removed link right_follower
- removed link right_pad
- removed link right_silicone_pad
- removed link right_spring_link
- added link 2f85-base, mass 0.777441; collision mesh filename=file:///workspace/model/ur5e_2f85/assets/base.stl scale=0.001 0.001 0.001; visual mesh filename=file:///workspace/model/ur5e_2f85/assets/base.stl scale=0.001 0.001 0.001
- added link base-mount; collision mesh filename=file:///workspace/model/ur5e_2f85/assets/base_mount.stl scale=0.001 0.001 0.001; visual mesh filename=file:///workspace/model/ur5e_2f85/assets/base_mount.stl scale=0.001 0.001 0.001
- added link left-coupler, mass 0.0140974; collision mesh filename=file:///workspace/model/ur5e_2f85/assets/coupler.stl scale=0.001 0.001 0.001; visual mesh filename=file:///workspace/model/ur5e_2f85/assets/coupler.stl scale=0.001 0.001 0.001
- added link left-driver, mass 0.00899563; collision mesh filename=file:///workspace/model/ur5e_2f85/assets/driver.stl scale=0.001 0.001 0.001; visual mesh filename=file:///workspace/model/ur5e_2f85/assets/driver.stl scale=0.001 0.001 0.001
- added link left-follower, mass 0.0125222; collision mesh filename=file:///workspace/model/ur5e_2f85/assets/follower.stl scale=0.001 0.001 0.001; visual mesh filename=file:///workspace/model/ur5e_2f85/assets/follower.stl scale=0.001 0.001 0.001
- added link left-pad, mass 0.0035; collision box size=0.022 0.008 0.01875; collision box size=0.022 0.008 0.01875
- added link left-silicone-pad; visual mesh filename=file:///workspace/model/ur5e_2f85/assets/silicone_pad.stl scale=0.001 0.001 0.001
- added link left-spring-link, mass 0.0221642; collision mesh filename=file:///workspace/model/ur5e_2f85/assets/spring_link.stl scale=0.001 0.001 0.001; visual mesh filename=file:///workspace/model/ur5e_2f85/assets/spring_link.stl scale=0.001 0.001 0.001
- added link pinch-site
- added link right-coupler, mass 0.0140974; collision mesh filename=file:///workspace/model/ur5e_2f85/assets/coupler.stl scale=0.001 0.001 0.001; visual mesh filename=file:///workspace/model/ur5e_2f85/assets/coupler.stl scale=0.001 0.001 0.001
- added link right-driver, mass 0.00899563; collision mesh filename=file:///workspace/model/ur5e_2f85/assets/driver.stl scale=0.001 0.001 0.001; visual mesh filename=file:///workspace/model/ur5e_2f85/assets/driver.stl scale=0.001 0.001 0.001
- added link right-follower, mass 0.0125222; collision mesh filename=file:///workspace/model/ur5e_2f85/assets/follower.stl scale=0.001 0.001 0.001; visual mesh filename=file:///workspace/model/ur5e_2f85/assets/follower.stl scale=0.001 0.001 0.001
- added link right-pad, mass 0.0035; collision box size=0.022 0.008 0.01875; collision box size=0.022 0.008 0.01875
- added link right-silicone-pad; visual mesh filename=file:///workspace/model/ur5e_2f85/assets/silicone_pad.stl scale=0.001 0.001 0.001
- added link right-spring-link, mass 0.0221642; collision mesh filename=file:///workspace/model/ur5e_2f85/assets/spring_link.stl scale=0.001 0.001 0.001; visual mesh filename=file:///workspace/model/ur5e_2f85/assets/spring_link.stl scale=0.001 0.001 0.001
Joints:
- joint 2f85_base_joint: child 2f85_base -> 2f85-base; parent base_mount -> base-mount
- joint base_mount_joint: child base_mount -> base-mount
- joint left_coupler_joint: child left_coupler -> left-coupler; mimic (none) -> joint=left_driver_joint multiplier=-1 offset=0; parent left_driver -> left-driver
- joint left_driver_joint: child left_driver -> left-driver; mimic (none) -> joint=right_driver_joint multiplier=1 offset=0; parent 2f85_base -> 2f85-base
- joint left_follower_joint: child left_follower -> left-follower; mimic (none) -> joint=left_driver_joint multiplier=-1 offset=0; parent left_spring_link -> left-spring-link
- joint left_pad_joint: child left_pad -> left-pad; parent left_follower -> left-follower
- joint left_silicone_pad_joint: child left_silicone_pad -> left-silicone-pad; parent left_pad -> left-pad
- joint left_spring_link_joint: child left_spring_link -> left-spring-link; mimic (none) -> joint=left_driver_joint multiplier=1 offset=0; parent 2f85_base -> 2f85-base
- joint pinch_site_joint: child pinch_site -> pinch-site; parent 2f85_base -> 2f85-base
- joint right_coupler_joint: child right_coupler -> right-coupler; mimic (none) -> joint=right_driver_joint multiplier=-1 offset=0; parent right_driver -> right-driver
- joint right_driver_joint: child right_driver -> right-driver; parent 2f85_base -> 2f85-base
- joint right_follower_joint: child right_follower -> right-follower; mimic (none) -> joint=right_driver_joint multiplier=-1 offset=0; parent right_spring_link -> right-spring-link
- joint right_pad_joint: child right_pad -> right-pad; parent right_follower -> right-follower
- joint right_silicone_pad_joint: child right_silicone_pad -> right-silicone-pad; parent right_pad -> right-pad
- joint right_spring_link_joint: child right_spring_link -> right-spring-link; mimic (none) -> joint=right_driver_joint multiplier=1 offset=0; parent 2f85_base -> 2f85-base

Commit message: ur5e origin z 수정

File: cobot_pnp_safety/urdf/ur5e_2f85.urdf (robot description, URDF)
Before this commit: robot ur5e_2f85, 24 links, 23 joints
Joints:
- joint virtual_joint: origin xyz=0 0 0 rpy=0 0 0 -> xyz=0 0 0.6 rpy=0 0 0

Commit message: assets 경로 수정

File: cobot_pnp_safety/urdf/ur5e_2f85.urdf (robot description, URDF)
Before this commit: robot ur5e_2f85, 24 links, 23 joints
Links:
- added link gripper_camera; visual box size=0.018 0.012 0.012
- added link gripper_camera_bracket
- added link gripper_camera_optical_frame
- link 2f85-base: geometry collision mesh filename=file:///workspace/assets/ur5e_2f85/base.stl scale=0.001 0.001 0.001; visual mesh filename=file:///workspace/assets/ur5e_2f85/base.stl scale=0.001 0.001 0.001
- link base: geometry visual mesh filename=file:///workspace/assets/ur5e_2f85/base_0.obj; visual mesh filename=file:///workspace/assets/ur5e_2f85/base_1.obj
- link base-mount: geometry collision mesh filename=file:///workspace/assets/ur5e_2f85/base_mount.stl scale=0.001 0.001 0.001; visual mesh filename=file:///workspace/assets/ur5e_2f85/base_mount.stl scale=0.001 0.001 0.001
- link forearm_link: geometry collision cylinder length=0.12 radius=0.055; collision cylinder length=0.38 radius=0.038
- link left-coupler: geometry collision mesh filename=file:///workspace/assets/ur5e_2f85/coupler.stl scale=0.001 0.001 0.001; visual mesh filename=file:///workspace/assets/ur5e_2f85/coupler.stl scale=0.001 0.001 0.001
- link left-driver: geometry collision mesh filename=file:///workspace/assets/ur5e_2f85/driver.stl scale=0.001 0.001 0.001; visual mesh filename=file:///workspace/assets/ur5e_2f85/driver.stl scale=0.001 0.001 0.001
- link left-follower: geometry collision mesh filename=file:///workspace/assets/ur5e_2f85/follower.stl scale=0.001 0.001 0.001; visual mesh filename=file:///workspace/assets/ur5e_2f85/follower.stl scale=0.001 0.001 0.001
- link left-pad: geometry collision box size=0.022 0.008 0.01875; collision box size=0.022 0.008 0.01875
- link left-silicone-pad: geometry visual mesh filename=file:///workspace/assets/ur5e_2f85/silicone_pad.stl scale=0.001 0.001 0.001
- link left-spring-link: geometry collision mesh filename=file:///workspace/assets/ur5e_2f85/spring_link.stl scale=0.001 0.001 0.001; visual mesh filename=file:///workspace/assets/ur5e_2f85/spring_link.stl scale=0.001 0.001 0.001
- link right-coupler: geometry collision mesh filename=file:///workspace/assets/ur5e_2f85/coupler.stl scale=0.001 0.001 0.001; visual mesh filename=file:///workspace/assets/ur5e_2f85/coupler.stl scale=0.001 0.001 0.001
- link right-driver: geometry collision mesh filename=file:///workspace/assets/ur5e_2f85/driver.stl scale=0.001 0.001 0.001; visual mesh filename=file:///workspace/assets/ur5e_2f85/driver.stl scale=0.001 0.001 0.001
- link right-follower: geometry collision mesh filename=file:///workspace/assets/ur5e_2f85/follower.stl scale=0.001 0.001 0.001; visual mesh filename=file:///workspace/assets/ur5e_2f85/follower.stl scale=0.001 0.001 0.001
- link right-pad: geometry collision box size=0.022 0.008 0.01875; collision box size=0.022 0.008 0.01875
- link right-silicone-pad: geometry visual mesh filename=file:///workspace/assets/ur5e_2f85/silicone_pad.stl scale=0.001 0.001 0.001
- link right-spring-link: geometry collision mesh filename=file:///workspace/assets/ur5e_2f85/spring_link.stl scale=0.001 0.001 0.001; visual mesh filename=file:///workspace/assets/ur5e_2f85/spring_link.stl scale=0.001 0.001 0.001
- link shoulder_link: geometry collision cylinder length=0.12 radius=0.06; visual mesh filename=file:///workspace/assets/ur5e_2f85/shoulder_0.obj
- link upper_arm_link: geometry collision cylinder length=0.12 radius=0.06; collision cylinder length=0.4 radius=0.05
- link wrist_1_link: geometry collision cylinder length=0.14 radius=0.04; visual mesh filename=file:///workspace/assets/ur5e_2f85/wrist1_0.obj
- link wrist_2_link: geometry collision cylinder length=0.08 radius=0.04; collision cylinder length=0.12 radius=0.04
- link wrist_3_link: geometry collision cylinder length=0.04 radius=0.04; visual mesh filename=file:///workspace/assets/ur5e_2f85/wrist3.obj
Joints:
- added joint gripper_camera_bracket_joint: type fixed, parent base-mount, child gripper_camera_bracket, origin xyz=0 -0.07 0 rpy=-1.74533 0 0
- added joint gripper_camera_joint: type fixed, parent gripper_camera_bracket, child gripper_camera, origin xyz=0 0 0.025 rpy=0 0 0
- added joint gripper_camera_optical_joint: type fixed, parent gripper_camera, child gripper_camera_optical_frame, origin xyz=0 0 0 rpy=3.14159265359 0 0
